File: pcb/tiltetcher/tiltetcher.kicad_sch (KiCad schematic)
At the start: 23 parts, among them J1 Jack-DC, J11 Screw_Terminal_01x02, J21 Screw_Terminal_01x07, J31 Screw_Terminal_01x07, K1 ADW11, M1 Motor_DC, Q1 IRF3205, SW1 SW_DIP_Main, SW2 SW_DIP_Motor, SW3 SW_DIP_HTR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

Commit message: heater works!
Connections:
- net HEATER: now also A1.18 (D3)
Changed lines of the file:
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@@
+    (stroke (width 0) (type default) (color 0 0 0 0))
+  )
+  (wire (pts (xy 21.59 95.25) (xy 45.72 95.25))
     (stroke (width 0) (type default) (color 0 0 0 0))
   )
@@
     (effects (font (size 1.27 1.27)) (justify left bottom))
   )
+  (label "HEATER" (at 21.59 95.25 0)
+    (effects (font (size 1.27 1.27)) (justify left bottom))
+  )
